File: PCBs/me_gizmo/me_gizmo.kicad_sch (KiCad schematic)
At the start: 47 parts, among them J5 DEBUG, J6 USB4105-GF-A, Q3 MBT3904DW1, U10 RP2350A, U13 MCP1702T-3302E_CB, U5 REF35250QDBVR, U6 TMP126-Q1, U7 TLV9152VSSOP, X1 IQXO-791

Commit message: Completed first draft of integrated measurement unit
Parts:
- removed D1: LED, LED_SMD:LED_0805_2012Metric, symbol Device:LED_Filled
- removed D2: IN-S85TATRGB, Eclectronics:IN-S85TATRGB, symbol Eclectronics:IN-S85TATRGB
- removed J5: DEBUG, Connector_PinHeader_2.54mm:PinHeader_1x03_P2.54mm_Vertical, symbol Connector_Generic:Conn_01x03
- removed Q3: MBT3904DW1, Package_TO_SOT_SMD:SOT-363_SC-70-6, symbol Transistor_BJT:MBT3904DW1
- removed R35, R45, R46: 1K, Resistor_SMD:R_0402_1005Metric, symbol Device:R
- removed R44: 5.1K, Resistor_SMD:R_0402_1005Metric, symbol Device:R
- removed U7: TLV9152VSSOP, Package_SO:VSSOP-8_3x3mm_P0.65mm, symbol Amplifier_Operational:TLV9152
- added C45: 0.1µF, Capacitor_SMD:C_0603_1608Metric, symbol Device:C
- added J5: Debug, Connector_PinHeader_2.54mm:PinHeader_1x04_P2.54mm_Vertical, symbol Connector_Generic:Conn_01x04
- added Q1: MMBT3904L, Package_TO_SOT_SMD:SOT-23, symbol Transistor_BJT:MMBT3904
- added R49: 10kΩ, Capacitor_SMD:C_0603_1608Metric, symbol Device:R
- added U8: TLV9151, Package_TO_SOT_SMD:SOT-23-5, symbol Eclectronics:MCP6021
- R28, R29: value 5.1K -> 5.1kΩ; footprint Resistor_SMD:R_0402_1005Metric -> Resistor_SMD:R_0603_1608Metric
- R30, R31: value 5.1K -> 5.1kΩ
- R47: value 1K -> 1kΩ; footprint Resistor_SMD:R_0402_1005Metric -> Resistor_SMD:R_0603_1608Metric
- R48: value 10k -> 10kΩ; footprint Resistor_SMD:R_0402_1005Metric -> Capacitor_SMD:C_0603_1608Metric
Connections:
- net GPIO22 is gone; now on net COPI: U10.34 (GPIO22)
- net GPIO24 is gone; now on net CIPO: U10.36 (GPIO24)
- net GPIO25 is gone; now on net TEMP_CS: U10.37 (GPIO25)
- net +3V3: now also C45.1, R49.2; no longer U10.17 (GPIO13), U6.5 (~{ALERT})
- net CIPO: no longer U10.27 (GPIO16)
- net COPI: no longer U10.31 (GPIO19)
- net GND: now also C45.2, J5.3 (Pin_3), U8.2
- net SCLK: now also U10.33 (GPIO21); no longer U10.29 (GPIO18)
- net SWCLK: now also J5.2 (Pin_2)
- net SWDIO: now also J5.4 (Pin_4)
- net TEMP_CS: no longer U10.16 (GPIO12)
- net VREF: now also U8.3
- net VREF_BUF: now also Q1.2 (E), U8.4
- net ~{DAC1_CS}: now also U10.31 (GPIO19); no longer U10.33 (GPIO21)
- net ~{DAC2_CS}: now also U10.32 (GPIO20); no longer U10.40 (GPIO26/ADC0)
- net ~{IRQ}/MDAT: now also U10.29 (GPIO18); no longer U10.32 (GPIO20)
- net ~{LDAC}: now also U10.27 (GPIO16); no longer U10.42 (GPIO28/ADC2)
- net GPIO11: now reaches U10.15 (GPIO11)
- net GPIO2: now reaches U10.4 (GPIO2)
- net GPIO2: now also J5.1 (Pin_1)
- net GPIO27: now reaches U10.41 (GPIO27/ADC1)
- net GPIO29: now reaches U10.43 (GPIO29/ADC3)
- net +5V renamed VBUS
- net VBUS: now also Q1.3 (C), U8.5
- net GPIO23 renamed TEMP_ALERT
- net TEMP_ALERT: now also U6.5 (~{ALERT}), R49.1
- new net: Q1.1 (B), U8.1
- new net GPIO26: U10.40 (GPIO26/ADC0)
- new net GPIO28: U10.42 (GPIO28/ADC2)
- no-connect marks 24 -> 22
Other:
- added sheet LEDs (LEDs.kicad_sch)
- moved on the sheet: C17, C18, C19, C2, C3, D3, R28, R29, R47, S1, S2, U13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

Commit message: Made a few final layout tweaks and added a BOM file
Parts:
- R30, R31: footprint Resistor_SMD:R_0402_1005Metric -> Resistor_SMD:R_0603_1608Metric
- R48, R49: footprint Capacitor_SMD:C_0603_1608Metric -> Resistor_SMD:R_0603_1608Metric
Changed lines of the file:
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@@
 			)
 		)
-		(property "Footprint" "Resistor_SMD:R_0402_1005Metric"
+		(property "Footprint" "Resistor_SMD:R_0603_1608Metric"
 			(at 51.562 48.26 90)
 			(effects
@@
 			)
 		)
-		(property "Footprint" "Resistor_SMD:R_0402_1005Metric"
+		(property "Footprint" "Resistor_SMD:R_0603_1608Metric"
 			(at 42.672 48.26 90)
 			(effects
@@
 			)
 		)
-		(property "Footprint" "Capacitor_SMD:C_0603_1608Metric"
+		(property "Footprint" "Resistor_SMD:R_0603_1608Metric"
 			(at 35.56 164.592 90)
 			(effects
@@
 			)
 		)
-		(property "Footprint" "Capacitor_SMD:C_0603_1608Metric"
+		(property "Footprint" "Resistor_SMD:R_0603_1608Metric"
 			(at 31.75 174.752 90)
 			(effects
